File: generated/pcbs/goose.kicad_pcb (KiCad board)
At the start: 2 copper layers, 132.2 x 96.8 mm, 42 parts

Commit message: partial
Parts:
- removed ?: , power_switch
- removed SW1: , sw_reset_side
- moved BAT1 15 test 17.5 mm to (271.5, 147.5), turned to -4.5 degrees
- moved D1 17.5 mm to (187.4, 169.4), turned to 96.5 degrees
- moved D2 17.5 mm to (185.2, 150.5), turned to 96.5 degrees
- moved D3 17.5 mm to (183.1, 131.6), turned to 96.5 degrees
- moved D19 17.5 mm to (284.9, 189.8), turned to 75.5 degrees
- moved D6 17.5 mm to (204.7, 122.7), turned to 92.5 degrees
- moved D4 17.5 mm to (206.4, 160.6), turned to 92.5 degrees
- moved D5 17.5 mm to (205.6, 141.7), turned to 92.5 degrees
- moved D10 17.5 mm to (246.3, 158.1), turned to 88.5 degrees
- moved D11 17.5 mm to (246.8, 139.1), turned to 88.5 degrees
- moved D12 17.5 mm to (247.3, 120.1), turned to 88.5 degrees
- moved D17 17.5 mm to (246.0, 177.7), turned to 88.5 degrees
- moved D18 17.5 mm to (265.2, 185.0), turned to 81.5 degrees
- moved D16 17.5 mm to (226.4, 174.1), turned to 90.5 degrees
- moved D8 17.5 mm to (226.1, 136.0), turned to 90.5 degrees
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Connections:
- net C0 renamed col_pinkie
- net C0_R0 renamed pinkie_top
- net C0_R1 renamed pinkie_home
- net C0_R2 renamed pinkie_bottom
- net C1 renamed col_ring
- net C1_R0 renamed ring_top
- net C1_R1 renamed ring_home
- net C1_R2 renamed ring_bottom
- net C1_R3 renamed middle_thumbs
- net C2 renamed col_middle
- net C2_R0 renamed middle_top
- net C2_R1 renamed middle_home
- net C2_R2 renamed middle_bottom
- net C2_R3 renamed inner_thumbs
- net C3 renamed col_index
- net C3_R0 renamed index_top
- net C3_R1 renamed index_home
- net C3_R2 renamed index_bottom
- net C3_R3 renamed outer_thumbs
- net C4 renamed col_inner
- net C4_R0 renamed inner_top
- net C4_R1 renamed inner_home
- net C4_R2 renamed inner_bottom
- net C4_R3 renamed reach_thumbs
- net R0 renamed row_top
- net R1 renamed row_home
- net R2 renamed row_bottom
- net R3 renamed row_thumb
- BAT1 15 test pad 1: BAT_P -> BATP
- BAT1 15 test pad 2: BAT- -> GND
- _1 pad : CLK -> RAW5V
Other:
- board size 132.2 x 96.8 mm -> 129.9 x 96.3 mm

Commit message: Almost finalized
Parts:
- removed BAT1 15 test: 18 line, BatteryPad
- added BAT1: , BatteryPad, F.Cu at (290.5, 137.8)
- added H1: , mounting_hole, F.Cu at (187.3, 132.2)
- added H2: , mounting_hole, F.Cu at (188.8, 151.1)
- added H3: , mounting_hole, F.Cu at (250.8, 118.7)
- added H4: , mounting_hole, F.Cu at (229.4, 163.0)
- added H5: , mounting_hole, F.Cu at (267.3, 169.5)
- added ROT1: , rotary_encoder, F.Cu at (282.2, 162.4)
- added SW1: , sw_reset_side, F.Cu at (261.7, 110.5)
- D1, D10, D11, D12, D13, D14, D15, D16, D17, D18, D19, D2, D3, D4, D5, D6, D7, D8, D9: footprint ComboDiode -> Diode_SMD:D_SOD-123; moved to F.Cu
- moved D3 14.0 mm to (169.2, 133.7), turned to 186.5 degrees
- moved D1 14.0 mm to (173.5, 171.5), turned to 186.5 degrees
- moved D2 14.0 mm to (171.4, 152.6), turned to 186.5 degrees
- moved D19 14.0 mm to (271.2, 186.8), turned to 165.5 degrees
- moved D18 14.0 mm to (251.3, 183.4), turned to 171.5 degrees
- moved D13 14.0 mm to (252.4, 163.6), turned to 177.5 degrees
- moved D14 14.0 mm to (253.2, 144.6), turned to 177.5 degrees
- moved D15 14.0 mm to (254.0, 125.7), turned to 177.5 degrees
- moved D4 14.0 mm to (192.4, 161.8), turned to 182.5 degrees
- moved D5 14.0 mm to (191.6, 142.8), turned to 182.5 degrees
- moved D6 14.0 mm to (190.8, 123.8), turned to 182.5 degrees
- moved D10 14.0 mm to (232.3, 158.2), turned to 178.5 degrees
- moved D11 14.0 mm to (232.8, 139.2), turned to 178.5 degrees
- moved D12 14.0 mm to (233.3, 120.2), turned to 178.5 degrees
- moved D17 14.0 mm to (232.0, 177.8), turned to 178.5 degrees
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Connections:
- net index_bottom renamed C3_R2
- net index_home renamed C3_R1
- net index_top renamed C3_R0
- net inner_bottom renamed C4_R2
- net inner_home renamed C4_R1
- net inner_thumbs renamed C2_R3
- net inner_top renamed C4_R0
- net middle_bottom renamed C2_R2
- net middle_home renamed C2_R1
- net middle_thumbs renamed C1_R3
- net middle_top renamed C2_R0
- net outer_thumbs renamed C3_R3
- net pinkie_bottom renamed C0_R2
- net pinkie_home renamed C0_R1
- net pinkie_top renamed C0_R0
- net reach_thumbs renamed C4_R3
- net ring_bottom renamed C1_R2
- net ring_home renamed C1_R1
- net ring_top renamed C1_R0
- D1 pad 1: row_bottom -> R2
- D10 pad 1: row_bottom -> R2
- D11 pad 1: row_home -> R1
- D12 pad 1: row_top -> R0
- D13 pad 1: row_bottom -> R2
- D14 pad 1: row_home -> R1
- D15 pad 1: row_top -> R0
- D16 pad 1: row_thumb -> R3
- D17 pad 1: row_thumb -> R3
- D18 pad 1: row_thumb -> R3
- D19 pad 1: row_thumb -> R3
- D2 pad 1: row_home -> R1
- D3 pad 1: row_top -> R0
- D4 pad 1: row_bottom -> R2
- D5 pad 1: row_home -> R1
- D6 pad 1: row_top -> R0
- D7 pad 1: row_bottom -> R2
- D8 pad 1: row_home -> R1
- D9 pad 1: row_top -> R0
- S1 pad 1: col_pinkie -> C0
- S10 pad 1: col_index -> C3
- S11 pad 1: col_index -> C3
- S12 pad 1: col_index -> C3
- S13 pad 1: col_inner -> C4
- S14 pad 1: col_inner -> C4
- S15 pad 1: col_inner -> C4
- S16 pad 1: col_ring -> C1
- S17 pad 1: col_middle -> C2
- S18 pad 1: col_index -> C3
- S19 pad 1: col_inner -> C4
- S2 pad 1: col_pinkie -> C0
- S3 pad 1: col_pinkie -> C0
- S4 pad 1: col_ring -> C1
- S5 pad 1: col_ring -> C1
- S6 pad 1: col_ring -> C1
- S7 pad 1: col_middle -> C2
- S8 pad 1: col_middle -> C2
- S9 pad 1: col_middle -> C2
- _1 pad : RAW5V -> CLK
- _1 pad 1: P0 -> R0
- _1 pad 10: P9 -> C3
- _1 pad 11: P10 -> C4
- _1 pad 2: P1 -> R1
- _1 pad 3: P2 -> R2
- _1 pad 4: P3 -> R3
- _1 pad 5: P4 -> C0
- _1 pad 6: P5 -> C1
- _1 pad 7: P6 -> C2
Other:
- board size 129.9 x 96.3 mm -> 131.7 x 96.3 mm
- board text added: "AN"
- board text added: "NEVER"
- board text added: "OPTION!"
- board text added: "PEACE"
- board text added: "WAS"
- board text added: "[BONK!]"

Commit message: Ok version
Parts:
- removed D1, D10, D11, D12, D13, D14, D15, D16, D17, D18, D19, D2, D3, D4, D5, D6, D7, D8, D9: , Diode_SMD:D_SOD-123
- removed SW1: , sw_reset_side
- removed _1: , Seeeduino XIAO nRF52840
- added ?: , Seeeduino XIAO nRF52840, F.Cu at (283.0, 125.9)
- added Di1: , Diode_SMD:D_SOD-123, B.Cu at (173.4, 170.5)
- added Di10: , Diode_SMD:D_SOD-123, B.Cu at (232.4, 157.2)
- added Di11: , Diode_SMD:D_SOD-123, B.Cu at (232.9, 138.2)
- added Di12: , Diode_SMD:D_SOD-123, B.Cu at (233.4, 119.2)
- added Di13: , Diode_SMD:D_SOD-123, B.Cu at (252.4, 162.6)
- added Di14: , Diode_SMD:D_SOD-123, B.Cu at (253.2, 143.6)
- added Di15: , Diode_SMD:D_SOD-123, B.Cu at (254.1, 124.7)
- added Di16: , Diode_SMD:D_SOD-123, B.Cu at (212.4, 173.7)
- added Di17: , Diode_SMD:D_SOD-123, B.Cu at (232.0, 176.8)
- added Di18: , Diode_SMD:D_SOD-123, B.Cu at (251.4, 182.4)
- added Di19: , Diode_SMD:D_SOD-123, B.Cu at (271.4, 185.8)
- added Di2: , Diode_SMD:D_SOD-123, B.Cu at (171.3, 151.6)
- added Di3: , Diode_SMD:D_SOD-123, B.Cu at (169.1, 132.7)
- added Di4: , Diode_SMD:D_SOD-123, B.Cu at (192.4, 160.8)
- added Di5: , Diode_SMD:D_SOD-123, B.Cu at (191.6, 141.8)
- added Di6: , Diode_SMD:D_SOD-123, B.Cu at (190.7, 122.8)
- added Di7: , Diode_SMD:D_SOD-123, B.Cu at (212.2, 154.6)
- added Di8: , Diode_SMD:D_SOD-123, B.Cu at (212.1, 135.6)
- added Di9: , Diode_SMD:D_SOD-123, B.Cu at (211.9, 116.6)
- added RSW1: , sw_reset_side, F.Cu at (261.7, 110.8)
- BAT1: moved to B.Cu
- moved BAT1 12.9 mm to (284.3, 126.5)
- moved ROT1 1.12 mm to (282.8, 161.4), turned to -2.5 degrees
- turned S1 to 6.5 degrees
- turned S10 to -1.5 degrees
- turned S11 to -1.5 degrees
- turned S12 to -1.5 degrees
- turned S13 to -2.5 degrees
- turned S14 to -2.5 degrees
- turned S15 to -2.5 degrees
- turned S16 to 0.5 degrees
- turned S17 to -1.5 degrees
- turned S18 to -8.5 degrees
- turned S19 to -14.5 degrees
- turned S2 to 6.5 degrees
- turned S3 to 6.5 degrees
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Connections:
- ROT1 pad A: P7 -> P0
- ROT1 pad B: P8 -> P1

Commit message: Mirrored pcbs
Parts:
- removed ?: , Seeeduino XIAO nRF52840
- removed RSW1: , sw_reset_side
- added BAT2: , BatteryPad, B.Cu at (281.1, 160.2)
- added Di20: , Diode_SMD:D_SOD-123, B.Cu at (384.1, 189.0)
- added Di21: , Diode_SMD:D_SOD-123, B.Cu at (384.1, 170.0)
- added Di22: , Diode_SMD:D_SOD-123, B.Cu at (384.1, 151.0)
- added Di23: , Diode_SMD:D_SOD-123, B.Cu at (364.2, 182.5)
- added Di24: , Diode_SMD:D_SOD-123, B.Cu at (362.9, 163.5)
- added Di25: , Diode_SMD:D_SOD-123, B.Cu at (361.5, 144.6)
- added Di26: , Diode_SMD:D_SOD-123, B.Cu at (343.8, 179.1)
- added Di27: , Diode_SMD:D_SOD-123, B.Cu at (341.8, 160.2)
- added Di28: , Diode_SMD:D_SOD-123, B.Cu at (339.9, 141.3)
- added Di29: , Diode_SMD:D_SOD-123, B.Cu at (324.2, 184.5)
- added Di30: , Diode_SMD:D_SOD-123, B.Cu at (321.5, 165.6)
- added Di31: , Diode_SMD:D_SOD-123, B.Cu at (318.9, 146.8)
- added Di32: , Diode_SMD:D_SOD-123, B.Cu at (304.9, 192.3)
- added Di33: , Diode_SMD:D_SOD-123, B.Cu at (301.9, 173.6)
- added Di34: , Diode_SMD:D_SOD-123, B.Cu at (299.0, 154.8)
- added Di35: , Diode_SMD:D_SOD-123, B.Cu at (345.9, 199.1)
- added Di36: , Diode_SMD:D_SOD-123, B.Cu at (326.7, 203.9)
- added Di37: , Diode_SMD:D_SOD-123, B.Cu at (308.4, 213.3)
- added Di38: , Diode_SMD:D_SOD-123, B.Cu at (289.4, 220.3)
- added H10: , mounting_hole, F.Cu at (301.7, 202.8)
- added H6: , mounting_hole, F.Cu at (380.0, 152.5)
- added H7: , mounting_hole, F.Cu at (380.7, 171.5)
- added H8: , mounting_hole, F.Cu at (336.7, 146.7)
- added H9: , mounting_hole, F.Cu at (341.7, 186.9)
- added ROT2: , rotary_encoder, F.Cu at (289.6, 191.2)
- added S20: , MX, F.Cu at (391.1, 184.5)
- added S21: , MX, F.Cu at (391.1, 165.5)
- added S22: , MX, F.Cu at (391.1, 146.5)
- added S23: , MX, F.Cu at (370.9, 177.5)
- added S24: , MX, F.Cu at (369.5, 158.5)
- added S25: , MX, F.Cu at (368.2, 139.6)
- added S26: , MX, F.Cu at (350.3, 173.9)
- added S27: , MX, F.Cu at (348.3, 155.0)
- added S28: , MX, F.Cu at (346.3, 136.1)
- added S29: , MX, F.Cu at (330.5, 179.0)
- added S30: , MX, F.Cu at (327.8, 160.2)
- added S31: , MX, F.Cu at (325.2, 141.4)
- added S32: , MX, F.Cu at (311.1, 186.8)
- added S33: , MX, F.Cu at (308.2, 168.0)
- added S34: , MX, F.Cu at (305.2, 149.3)
- added S35: , MX, F.Cu at (352.4, 193.9)
- added S36: , MX, F.Cu at (333.0, 198.4)
- added S37: , MX, F.Cu at (314.0, 207.1)
- added S38: , MX, F.Cu at (294.3, 213.6)
- added _1: , Seeeduino XIAO nRF52840, F.Cu at (257.0, 156.7)
- added _2: , Seeeduino XIAO nRF52840, F.Cu at (284.1, 156.7)
- moved H3 54.2 mm to (204.4, 146.7), turned to -7 degrees
- moved BAT1 45.1 mm to (253.1, 159.1), turned to -9 degrees
- moved S19 44.6 mm to (246.8, 213.6), turned to -21 degrees
- moved Di19 44.1 mm to (238.7, 215.3), turned to 69 degrees
- moved H5 43.4 mm to (239.4, 202.8), turned to -18 degrees
- moved ROT1 43.1 mm to (251.6, 191.2), turned to 261 degrees
- moved S18 42.6 mm to (227.1, 207.1), turned to -15 degrees
- moved Di18 42.3 mm to (219.2, 209.7), turned to 75 degrees
- moved S13 41.0 mm to (230.0, 186.8), turned to -9 degrees
- moved Di13 40.7 mm to (222.4, 190.1), turned to 81 degrees
- moved S17 40.5 mm to (208.1, 198.4), turned to -8 degrees
- moved Di17 40.3 mm to (200.5, 201.9), turned to 82 degrees
- moved S14 39.6 mm to (233.0, 168.0), turned to -9 degrees
- moved S16 39.4 mm to (188.7, 193.9), turned to -6 degrees
- moved Di14 39.3 mm to (225.3, 171.4), turned to 81 degrees
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Connections:
- BAT1 pad 1: BAT+ -> BATP
- BAT1 pad 2: BAT- -> GND
- ROT1 pad A: P0 -> RA
- ROT1 pad B: P1 -> RB
Other:
- board size 131.7 x 96.3 mm -> 266.1 x 106.6 mm
- board text added: "!#@"
- board text added: "JLCJLCJLCJLC"
- board text added: "gooses v0.8a"
- board text added: "↑gås upp↑"
- board text added: "↓gås ner↓"
- board text removed: "AN"
- board text removed: "NEVER"
- board text removed: "OPTION!"
- board text removed: "PEACE"
- board text removed: "WAS"
- board text removed: "[BONK!]"
